File: electrical hardware/kicad/magic dial/magic dial/magic dial.kicad_sch (KiCad schematic)
At the start: 14 parts, among them J1 GSB3C3133DS2HR, U2 CH224K, U3 TMC6300-LA-T, U4 MAQ430GQE-AEC1-Z, U5 INA240A1QPWRQ1, U6 ESP32-C6-WROOM-1-N8, U8 TLV75733PDBVR

Commit message: Major Update: Added Power, and Motor to Schematics
Major Update: Added Power, and Motor to Schematics
Parts:
- added C1, C3, C4: 0.1u, symbol Device:C_Small
- added C2: 22u, symbol Device:C_Small
- added C5, C6: 1u, symbol Device:C_Small
- added C7: 10u_Tan, symbol Device:C_Polarized_Small_US
- added C8: 10u, symbol Device:C_Polarized_Small_US
- added C9: 47u, symbol Device:C_Polarized_Small_US
- added J2: JST_CONN_01x03_PIN, symbol Connector:Conn_01x03_Pin
- added R10, R11, R12, R13, R8, R9: 100k, symbol Device:R_Small
- added R14, R15, R16, R7: 0.012, symbol Device:R_Small
- added R6: 10k, symbol Device:R_Small
Connections:
- net VBUS is gone; now on net VBUS_9V: J1.A4 (VBUS_A), J1.A9 (VBUS_A__1), J1.B4 (VBUS_B), J1.B9 (VBUS_B__1), R1.1, R2.1, VR1.3 (INPUT)
- net GND: now also J1.A1 (GND_A), J1.A12 (GND_A__1), J1.B1 (GND_B), U3.14 (GND), U3.21 (GND), U3.8 (GND), U3.9 (GND), C1.2, C2.2, C3.2, C5.2, C6.2, C7.2, C8.2, C9.2, R10.1, R11.1, R12.1, R13.1, R7.1, R8.1, R9.1
- net VDD: no longer R1.2, U2.1 (VDD), U6.2 (3V3), U8.5 (OUT)
- net VCC_5V: now reaches U8.1 (IN), U8.3 (EN), VR1.2 (OUTPUT_2), VR1.4 (OUTPUT_4)
- net VCC_5V: now also C6.1, C7.1
- net TMC6300_W: now reaches U3.1 (W)
- net TMC6300_W: now also R14.2
- net TMC6300_VL: now reaches U3.10 (VL)
- net TMC6300_VL: now also U6.26 (IO3), R13.2
- net VDD_3V3: now reaches U3.11 (VIO/NSTDBY)
- net VDD_3V3: now also R1.2, U2.1 (VDD), U6.2 (3V3), U8.5 (OUT), C1.1, C2.1, C4.1, C5.1, R6.2
- net TMC6300_DIAG: now reaches U3.12 (DIAG)
- net +1V8: now reaches U3.13 (1.8VOUT)
- net +1V8: now also C3.1
- net TMC6300_U: now reaches U3.15 (U)
- net TMC6300_U: now also R16.2
- net MCP6021_SENSE: now reaches U3.16 (BRUV)
- net MCP6021_SENSE: now also U3.20 (BRW), R7.2
- net TMC6300_V: now reaches U3.17 (V)
- net TMC6300_V: now also R15.2
- net VBUS_9V: now reaches U3.18 (VS)
- net VBUS_9V: now also C8.1, C9.1
- net TMC6300_VCP: now reaches U3.2 (VCP)
- net TMC6300_VCP: now also C4.2
- net TMC6300_UH: now reaches U3.3 (UH)
- net TMC6300_UH: now also U6.8 (IO0), R12.2
- net TMC6300_VH: now reaches U3.4 (VH)
- net TMC6300_VH: now also U6.27 (IO2), R11.2
- net TMC6300_WH: now reaches U3.5 (WH)
- net TMC6300_WH: now also U6.4 (IO4), R10.2
- net TMC6300_UL: now reaches U3.6 (UL)
- net TMC6300_UL: now also U6.9 (IO1), R9.2
- net TMC6300_WL: now reaches U3.7 (WL)
- net TMC6300_WL: now also U6.5 (IO5), R8.2
- net ESP32_BOOTMODE: now reaches U6.10 (IO8)
- net USB_DN: now reaches U6.13 (IO12)
- net USB_DN: now also J1.A7 (DN1), J1.B7 (DN2), U2.5 (DM)
- net USB_DP: now reaches U6.14 (IO13)
- net USB_DP: now also J1.A6 (DP1), J1.B6 (DP2), U2.4 (DP)
- net ESP32_JTAG: now reaches U6.15 (IO9)
- net ESP32_JTAG: now also U6.23 (IO15)
- net ESP32_SDA: now reaches U6.19 (IO21)
- net ESP32_SCL: now reaches U6.20 (IO22)
- net ESP32_RST: now reaches U6.3 (EN)
- net ESP32_RST: now also R6.1
- net CC1 renamed USB_CC1
- net CC2 renamed USB_CC2
- removed net DN: J1.A7 (DN1), J1.B7 (DN2), U2.5 (DM), U6.16 (IO18)
- removed net DP: J1.A6 (DP1), J1.B6 (DP2), U2.4 (DP), U6.17 (IO19)
- new net INA_U: J2.3 (Pin_3), R16.1
- new net INA_V: J2.2 (Pin_2), R15.1
- new net INA_W: J2.1 (Pin_1), R14.1
Other:
- note added: "Input Buttons"
- note added: "LED's"
- note added: "Load Cell: HX711"
- note added: "Microcontroller"
- note added: "Motor Current Sense"
- note added: "Motor: Max 2.8A"
- note added: "Power System: 9V 5A - 5V 3A - 3.3V 1A - 1.8V 5mA"
- note added: "Pull-Up/Down"
- note added: "Screen"
- note added: "Test Points"
- note removed: "5V and 3.3V LDO"
- company: (none) -> https://github.com/10-Percent-Complete/magic-dial
- title: (none) -> Magic Dial
- moved on the sheet: D1, R1, R2, R3, R4, R5, U2, U3, U4, U5, U8
