File: electrical hardware/kicad/magic dial/magic dial.kicad_pcb (KiCad board)
At the start: 2 copper layers, 1.6 x 9.2 mm, 63 parts, among them J1 GSB3C3133DS2HR, J2 MOTOR_JST_CONN_01x03_PIN, J3 Motor Power, J4 i2C Connector, J5 External_5V, J6 Bootmode Button, J7 RST Button, J8 UART Connector, J9 SPI Screen Connector, U1 INA240A1QPWRQ1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

Commit message: Auto Route Progress: Incomplete.
Auto Route Progress: Incomplete.
Parts:
- moved U5 2.82 mm to (107.7, 118.0)
- moved R14 2.82 mm to (130.5, 118.0)
- moved R2 2.82 mm to (117.5, 118.0)
- moved R3 2.82 mm to (124.2, 118.0)
- moved R13 2.36 mm to (150.5, 118.3)
- moved R11 2.36 mm to (145.1, 118.3)
- moved J1 0.14 mm to (53.1, 95.3)
- turned C6 to 180 degrees
Connections:
- C6 pad 1: +9V -> TMC6300_VS
- C6 pad 2: +9V -> TMC6300_VCP
Routing:
- net VDD_3V3: track 0.00 -> 177.2 mm, vias 0 -> 1
- net INA_W: track 0.00 -> 133.3 mm
- net TMC6300_VL: track 0.00 -> 120.2 mm, vias 0 -> 3
- net TMC6300_VH: track 0.00 -> 112.6 mm, vias 0 -> 4
- net ESP32_SCK: track 0.00 -> 111.8 mm, vias 0 -> 3
- net ESP32_MISO: track 0.00 -> 109.4 mm, vias 0 -> 2
- net TMC6300_UH: track 0.00 -> 108.3 mm, vias 0 -> 4
- net INA_V: track 0.00 -> 107.7 mm
- net ESP32_CS: track 0.00 -> 107.6 mm, vias 0 -> 2
- net TMC6300_WL: track 0.00 -> 105.5 mm, vias 0 -> 5
- net ESP32_RST: track 0.00 -> 104.7 mm, vias 0 -> 3
- net ESP32_MOSI: track 0.00 -> 102.7 mm, vias 0 -> 2
- net TMC6300_WH: track 0.00 -> 98.6 mm, vias 0 -> 4
- net MAQ_VDD: track 0.00 -> 95.0 mm, vias 0 -> 2
- net INA_U: track 0.00 -> 91.6 mm
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- added copper zone on B.Cu, net GND
- added copper zone on F.Cu, net GND
Other:
- board size 1.6 x 9.2 mm -> 117.1 x 77.2 mm
