File: electrical hardware/kicad/magic dial/magic dial.kicad_sch (KiCad schematic)
At the start: 60 parts, among them J1 GSB3C3133DS2HR, J10 RST Button, J2 MOTOR_JST_CONN_01x03_PIN, J3 Motor Power, J4 External_5V, J5 UART Connector, J6 i2C Connector, J7 SPI Screen Connector, J9 Bootmode Button, U1 INA240A1QPWRQ1, U2 INA240A1QPWRQ1, U3 TMC6300-LA-T, U4 MAQ430GQE-AEC1-Z, U5 INA240A1QPWRQ1, U6 ESP32-C6-WROOM-1-N8, U7 MCP6021T-E_OT, U8 TLV75733PDBVR

Commit message: Completed Validation or Schematic. Removed Errors. Needs Footprint assignment
Parts:
- added NT1, NT2, NT3: NetTie_2, symbol Device:NetTie_2
Connections:
- net +1V8: now also NT2.2; no longer U3.13 (1.8VOUT)
- net +9V: now also NT1.1, NT3.1; no longer C9.1, U3.18 (VS), U3.2 (VCP)
- net GND: now also C10.1
- net INA240_U_OUT: no longer U2.8 (OUT), U5.8 (OUT)
- net INA240_V_OUT: now also U2.8 (OUT)
- net INA240_W_OUT: now also U5.8 (OUT)
- net INA_V: no longer U5.3 (IN-)
- net INA_W: now also U5.3 (IN-)
- net MAQ_VDD: now also C10.2, U4.13 (VDD); no longer C10.1
- net TMC6300_V: no longer U5.2 (IN+)
- net TMC6300_W: now also U5.2 (IN+)
- net ESP32_JTAG: no longer names the net of U6.23 (IO15)
- net USB_CC1: no longer names the net of J1.A5 (CC1)
- net USB_CC2: no longer names the net of J1.B5 (CC2)
- new net TMC6300_1.8V: NT2.1, U3.13 (1.8VOUT)
- new net TMC6300_VCP: NT1.2, U3.2 (VCP)
- new net TMC6300_VS: C9.1, NT3.2, U3.18 (VS)
- no-connect marks 27 -> 29
Other:
- moved on the sheet: C10, C3, C4, C9, J4

Commit message: Assigned footprints for universal components. Need to do custom Components
Assigned footprints for universal components. Need to do custom Components
Parts:
- C1: renamed from C6; footprint (none) -> Capacitor_SMD:C_1206_3216Metric
- C2: renamed from C5; footprint (none) -> Capacitor_SMD:C_1206_3216Metric
- C3: renamed from C1; footprint (none) -> Capacitor_SMD:C_1206_3216Metric
- C4: renamed from C2; footprint (none) -> Capacitor_SMD:C_1206_3216Metric
- C5: renamed from C10; footprint (none) -> Capacitor_SMD:C_1206_3216Metric
- C6: renamed from C4; footprint (none) -> Capacitor_SMD:C_1206_3216Metric
- C7: renamed from C9; footprint (none) -> Capacitor_SMD:C_1206_3216Metric
- C8: renamed from C3; footprint (none) -> Capacitor_SMD:C_1206_3216Metric
- D1, D2, D3, D4, D5: footprint (none) -> LED_SMD:LED_1206_3216Metric
- J2: footprint (none) -> Connector_JST:JST_GH_SM03B-GHS-TB_1x03-1MP_P1.25mm_Horizontal
- J3: footprint (none) -> Connector_PinHeader_2.54mm:PinHeader_1x02_P2.54mm_Vertical
- J4: renamed from J6; footprint (none) -> Connector_PinHeader_2.54mm:PinHeader_1x04_P2.54mm_Vertical
- J5: renamed from J4; footprint (none) -> Connector_PinHeader_2.54mm:PinHeader_1x02_P2.54mm_Vertical
- J6: renamed from J9; footprint (none) -> Connector_PinHeader_2.54mm:PinHeader_1x02_P2.54mm_Vertical
- J7: renamed from J10; footprint (none) -> Connector_PinHeader_2.54mm:PinHeader_1x02_P2.54mm_Vertical
- J8: renamed from J5; footprint (none) -> Connector_PinHeader_2.54mm:PinHeader_1x05_P2.54mm_Vertical
- J9: renamed from J7; footprint (none) -> Connector_PinHeader_2.54mm:PinHeader_1x06_P2.54mm_Vertical
- NT1: footprint (none) -> NetTie:NetTie-2_SMD_Pad0.5mm
- NT2: renamed from NT3; footprint (none) -> NetTie:NetTie-2_SMD_Pad0.5mm
- NT3: renamed from NT2; footprint (none) -> NetTie:NetTie-2_SMD_Pad0.5mm
- R1: renamed from R6; footprint (none) -> Resistor_SMD:R_1206_3216Metric
- R10: renamed from R16; footprint (none) -> Resistor_SMD:R_1206_3216Metric
- R11, R12, R13: footprint (none) -> Resistor_SMD:R_1206_3216Metric
- R14: renamed from R7; footprint (none) -> Resistor_SMD:R_1206_3216Metric
- R15: renamed from R25; footprint (none) -> Resistor_SMD:R_1206_3216Metric
- R16: renamed from R26; footprint (none) -> Resistor_SMD:R_1206_3216Metric
- R17: renamed from R27; footprint (none) -> Resistor_SMD:R_1206_3216Metric
- R18: renamed from R28; footprint (none) -> Resistor_SMD:R_1206_3216Metric
- R19: renamed from R29; footprint (none) -> Resistor_SMD:R_1206_3216Metric
- R2: renamed from R18; footprint (none) -> Resistor_SMD:R_1206_3216Metric
- R20: renamed from R30; footprint (none) -> Resistor_SMD:R_1206_3216Metric
- R21: renamed from R19; footprint (none) -> Resistor_SMD:R_1206_3216Metric
- R22: renamed from R4; footprint (none) -> Resistor_SMD:R_1206_3216Metric
- R23: renamed from R5; footprint (none) -> Resistor_SMD:R_1206_3216Metric
- R24: renamed from R20; footprint (none) -> Resistor_SMD:R_1206_3216Metric
- R25: renamed from R21; footprint (none) -> Resistor_SMD:R_1206_3216Metric
- R26: renamed from R22; footprint (none) -> Resistor_SMD:R_1206_3216Metric
- R27: renamed from R23; footprint (none) -> Resistor_SMD:R_1206_3216Metric
- R28: renamed from R2; footprint (none) -> Resistor_SMD:R_1206_3216Metric
- R29: renamed from R24; footprint (none) -> Resistor_SMD:R_1206_3216Metric
- R3: renamed from R17; footprint (none) -> Resistor_SMD:R_1206_3216Metric
- R30: renamed from R3; footprint (none) -> Resistor_SMD:R_1206_3216Metric
- R4: renamed from R1; footprint (none) -> Resistor_SMD:R_1206_3216Metric
- R5: renamed from R8; footprint (none) -> Resistor_SMD:R_1206_3216Metric
- R6: renamed from R14; footprint (none) -> Resistor_SMD:R_1206_3216Metric
- R7: renamed from R9; footprint (none) -> Resistor_SMD:R_1206_3216Metric
- R8: renamed from R15; footprint (none) -> Resistor_SMD:R_1206_3216Metric
- R9: renamed from R10; footprint (none) -> Resistor_SMD:R_1206_3216Metric
- renumbered U5 to U2, U6 to U3, U2 to U4, U7 to U5, U3 to U6, U8 to U7, U4 to U8

Commit message: Completed Initial Layout for PCB
Parts:
- U1, U2, U4: footprint PW0008A_N -> INA240A1QPWRQ1:PW0008A_M
- U3: footprint ESP32-C6-WROOM-1-N8:XCVR_ESP32-C6-WROOM-1-N8 -> ESP32_C6_WROOM_1_N8:XCVR_ESP32-C6-WROOM-1-N8
- U5: footprint MCP6021T-E_OT:SOT95P270X145-5N -> MCP6021T_E_OT:SOT95P270X145-5N
- U6: footprint 21-100586_K2033+1C_ADI -> TMC6300_LA_T:21-100586_K2033&plus_1C_ADI-M
- U8: footprint QFN-16_MAQ430 -> MAQ430GQE_AEC1_Z:QFN-16_MAQ430-M
Changed lines of the file:
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@@
 			)
 		)
-		(property "Footprint" "21-100586_K2033+1C_ADI"
+		(property "Footprint" "TMC6300_LA_T:21-100586_K2033&plus_1C_ADI-M"
 			(at 157.48 96.52 0)
 			(effects
@@
 			)
 		)
-		(property "Footprint" "PW0008A_N"
+		(property "Footprint" "INA240A1QPWRQ1:PW0008A_M"
 			(at 58.42 222.25 0)
 			(effects
@@
 			)
 		)
-		(property "Footprint" "QFN-16_MAQ430"
+		(property "Footprint" "MAQ430GQE_AEC1_Z:QFN-16_MAQ430-M"
 			(at 223.52 243.84 0)
 			(effects
@@
 			)
 		)
-		(property "Footprint" "PW0008A_N"
+		(property "Footprint" "INA240A1QPWRQ1:PW0008A_M"
 			(at 127 222.25 0)
 			(effects
@@
 			)
 		)
-		(property "Footprint" "MCP6021T-E_OT:SOT95P270X145-5N"
+		(property "Footprint" "MCP6021T_E_OT:SOT95P270X145-5N"
 			(at 130.81 252.73 0)
 			(effects
@@
 			)
 		)
-		(property "Footprint" "ESP32-C6-WROOM-1-N8:XCVR_ESP32-C6-WROOM-1-N8"
+		(property "Footprint" "ESP32_C6_WROOM_1_N8:XCVR_ESP32-C6-WROOM-1-N8"
 			(at 59.69 128.27 0)
 			(effects
@@
 			)
 		)
-		(property "Footprint" "PW0008A_N"
+		(property "Footprint" "INA240A1QPWRQ1:PW0008A_M"
 			(at 58.42 257.81 0)
 			(effects

Commit message: Auto Route Progress: Incomplete.
Auto Route Progress: Incomplete.
Connections:
- net +9V: no longer C6.1, C6.2
- net TMC6300_VCP: now also C6.2
- net TMC6300_VS: now also C6.1
Other:
- moved on the sheet: C6, NT1, NT2
Changed lines of the file:
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@@
 	)
 	(junction
+		(at 346.71 60.96)
+		(diameter 0)
+		(color 0 0 0 0)
+	)
+	(junction
 		(at 400.05 50.8)
 		(diameter 0)
@@
 	)
 	(junction
-		(at 344.17 41.91)
-		(diameter 0)
-		(color 0 0 0 0)
-	)
-	(junction
-		(at 344.17 60.96)
-		(diameter 0)
-		(color 0 0 0 0)
-	)
-	(junction
 		(at 130.81 46.99)
 		(diameter 0)
@@
 	)
 	(junction
+		(at 346.71 41.91)
+		(diameter 0)
+		(color 0 0 0 0)
+	)
+	(junction
 		(at 113.03 266.7)
 		(diameter 0)
@@
 	(wire
 		(pts
-			(xy 344.17 41.91) (xy 344.17 48.26)
-		)
-		(stroke
-			(width 0)
-			(type default)
-		)
-	)
-	(wire
-		(pts
 			(xy 389.89 38.1) (xy 389.89 50.8)
 		)
@@
 	(wire
 		(pts
-			(xy 337.82 60.96) (xy 344.17 60.96)
-		)
-		(stroke
-			(width 0)
-			(type default)
-		)
-	)
-	(wire
-		(pts
 			(xy 359.41 194.31) (xy 367.03 194.31)
 		)
@@
 	(wire
 		(pts
+			(xy 346.71 60.96) (xy 351.79 60.96)
+		)
+		(stroke
+			(width 0)
+			(type default)
+		)
+	)
+	(wire
+		(pts
 			(xy 355.6 201.93) (xy 359.41 201.93)
 		)
@@
 	(wire
 		(pts
-			(xy 350.52 60.96) (xy 351.79 60.96)
+			(xy 344.17 60.96) (xy 346.71 60.96)
 		)
 		(stroke
@@
 	(wire
 		(pts
-			(xy 337.82 41.91) (xy 344.17 41.91)
+			(xy 337.82 41.91) (xy 340.36 41.91)
 		)
 		(stroke
@@
 	(wire
 		(pts
-			(xy 344.17 60.96) (xy 345.44 60.96)
+			(xy 337.82 60.96) (xy 339.09 60.96)
 		)
 		(stroke
@@
 	(wire
 		(pts
+			(xy 346.71 41.91) (xy 346.71 48.26)
+		)
+		(stroke
+			(width 0)
+			(type default)
+		)
+	)
+	(wire
+		(pts
 			(xy 271.78 49.53) (xy 312.42 49.53)
 		)
@@
 	(wire
 		(pts
-			(xy 344.17 41.91) (xy 347.98 41.91)
-		)
-		(stroke
-			(width 0)
-			(type default)
-		)
-	)
-	(wire
-		(pts
 			(xy 334.01 109.22) (xy 334.01 113.03)
 		)
@@
 	(wire
 		(pts
+			(xy 346.71 53.34) (xy 346.71 60.96)
+		)
+		(stroke
+			(width 0)
+			(type default)
+		)
+	)
+	(wire
+		(pts
 			(xy 281.94 100.33) (xy 281.94 113.03)
 		)
@@
 	(wire
 		(pts
-			(xy 353.06 41.91) (xy 356.87 41.91)
+			(xy 345.44 41.91) (xy 346.71 41.91)
 		)
 		(stroke
@@
 	(wire
 		(pts
-			(xy 344.17 53.34) (xy 344.17 60.96)
+			(xy 177.8 158.75) (xy 177.8 161.29)
 		)
 		(stroke
@@
 	(wire
 		(pts
-			(xy 177.8 158.75) (xy 177.8 161.29)
+			(xy 208.28 172.72) (xy 214.63 172.72)
 		)
 		(stroke
@@
 	(wire
 		(pts
-			(xy 208.28 172.72) (xy 214.63 172.72)
+			(xy 346.71 41.91) (xy 356.87 41.91)
 		)
 		(stroke
@@
 	(symbol
 		(lib_id "Device:C_Small")
-		(at 344.17 50.8 0)
+		(at 346.71 50.8 0)
 		(unit 1)
 		(exclude_from_sim no)
@@
 		(fields_autoplaced yes)
 		(property "Reference" "C6"
-			(at 346.71 49.5362 0)
+			(at 349.25 49.5362 0)
 			(effects
 				(font
@@
 		)
 		(property "Value" "100n"
-			(at 346.71 52.0762 0)
+			(at 349.25 52.0762 0)
 			(effects
 				(font
@@
 		)
 		(property "Footprint" "Capacitor_SMD:C_1206_3216Metric"
-			(at 344.17 50.8 0)
+			(at 346.71 50.8 0)
 			(effects
 				(font
@@
 		)
 		(property "Datasheet" "~"
-			(at 344.17 50.8 0)
+			(at 346.71 50.8 0)
 			(effects
 				(font
@@
 		)
 		(property "Description" "Unpolarized capacitor, small symbol"
-			(at 344.17 50.8 0)
+			(at 346.71 50.8 0)
 			(effects
 				(font
@@
 	(symbol
 		(lib_id "Device:NetTie_2")
-		(at 347.98 60.96 0)
+		(at 341.63 60.96 0)
 		(unit 1)
 		(exclude_from_sim no)
@@
 		(dnp no)
 		(property "Reference" "NT1"
-			(at 345.948 65.786 0)
+			(at 339.598 65.786 0)
 			(effects
 				(font
@@
 		)
 		(property "Value" "NetTie_2"
-			(at 345.948 63.754 0)
+			(at 339.598 63.5 0)
 			(effects
 				(font
@@
 		)
 		(property "Footprint" "NetTie:NetTie-2_SMD_Pad0.5mm"
-			(at 347.98 60.96 0)
+			(at 341.63 60.96 0)
 			(effects
 				(font
@@
 		)
 		(property "Datasheet" "~"
-			(at 347.98 60.96 0)
+			(at 341.63 60.96 0)
 			(effects
 				(font
@@
 		)
 		(property "Description" "Net tie, 2 pins"
-			(at 347.98 60.96 0)
+			(at 341.63 60.96 0)
 			(effects
 				(font
@@
 	(symbol
 		(lib_id "Device:NetTie_2")
-		(at 350.52 41.91 0)
+		(at 342.9 41.91 0)
 		(unit 1)
 		(exclude_from_sim no)
@@
 		(fields_autoplaced yes)
 		(property "Reference" "NT2"
-			(at 350.52 36.83 0)
+			(at 342.9 36.83 0)
 			(effects
 				(font
@@
 		)
 		(property "Value" "NetTie_2"
-			(at 350.52 39.37 0)
+			(at 342.9 39.37 0)
 			(effects
 				(font
@@
 		)
 		(property "Footprint" "NetTie:NetTie-2_SMD_Pad0.5mm"
-			(at 350.52 41.91 0)
+			(at 342.9 41.91 0)
 			(effects
 				(font
@@
 		)
 		(property "Datasheet" "~"
-			(at 350.52 41.91 0)
+			(at 342.9 41.91 0)
 			(effects
 				(font
@@
 		)
 		(property "Description" "Net tie, 2 pins"
-			(at 350.52 41.91 0)
+			(at 342.9 41.91 0)
 			(effects
 				(font
